File: uac.sch (EAGLE design)
At the start: 206 parts, among them Q6 2N7002CK4SST, Q7 2N7002CK4SST, U2 ADXL345, Y1 RESONATORSMD

Commit message: connecting
Parts:
- removed C10, C12, C13, C14, C15, C9: 100n, Custom components:C-EUC0603
Connections:
- net +3V3: no longer C10.1, C12.1, C13.1, C14.1, C15.1, C9.1
- net GND: now also U$1.BOOT0, U$1.PB2; no longer C10.2, C12.2, C13.2, C14.2, C15.2, C9.2
- net N$1: now also U$1.PD1-OSC_OUT
- net N$2: now also U$1.PD0-OSC_IN
- net RST: now also U$1.NRST
- net TCK: now also U$1.PA14
- net TDO: now also U$1.PB3
- net TMS: now also U$1.PA13
- net TRST: now also U$1.PB4
Other:
- moved on the sheet: R16, Y1
Changed lines of the file:
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@@
 <part name="+3V7" library="supply1" deviceset="+3V3" device=""/>
 <part name="R16" library="Custom components" deviceset="R-EU_" device="R0603" value="10k"/>
-<part name="C9" library="Custom components" deviceset="C-EU" device="C0603" value="100n"/>
-<part name="C10" library="Custom components" deviceset="C-EU" device="C0603" value="100n"/>
-<part name="C12" library="Custom components" deviceset="C-EU" device="C0603" value="100n"/>
-<part name="C13" library="Custom components" deviceset="C-EU" device="C0603" value="100n"/>
-<part name="C14" library="Custom components" deviceset="C-EU" device="C0603" value="100n"/>
-<part name="C15" library="Custom components" deviceset="C-EU" device="C0603" value="100n"/>
 <part name="GND4" library="supply1" deviceset="GND" device=""/>
 <part name="C18" library="Custom components" deviceset="C-EU" device="C0603" value="100n"/>
@@
 <part name="JP1" library="SparkFun2012" deviceset="JUMPER-2" device="SMD-NO"/>
 <part name="U$1" library="stm32" deviceset="STM32F103CBT6" device=""/>
+<part name="GND3" library="Custom components" deviceset="GND" device=""/>
+<part name="GND5" library="Custom components" deviceset="GND" device=""/>
 </parts>
 <sheets>
@@
 <instance part="C4" gate="G$1" x="147.32" y="215.9"/>
 <instance part="+3V2" gate="G$1" x="132.08" y="223.52"/>
-<instance part="Y1" gate="G$1" x="325.12" y="218.44" rot="R270"/>
-<instance part="GND2" gate="1" x="314.96" y="213.36"/>
+<instance part="Y1" gate="G$1" x="127" y="320.04" rot="R270"/>
+<instance part="GND2" gate="1" x="116.84" y="314.96"/>
 <instance part="MASTER_PROG" gate="A" x="35.56" y="203.2"/>
 <instance part="GND19" gate="1" x="12.7" y="208.28"/>
@@
 <instance part="+3V5" gate="G$1" x="154.94" y="401.32"/>
 <instance part="GND9" gate="1" x="154.94" y="299.72"/>
-<instance part="+3V7" gate="G$1" x="200.66" y="218.44"/>
-<instance part="R16" gate="G$1" x="208.28" y="213.36" rot="R180"/>
-<instance part="C9" gate="G$1" x="152.4" y="215.9"/>
-<instance part="C10" gate="G$1" x="157.48" y="215.9"/>
-<instance part="C12" gate="G$1" x="162.56" y="215.9"/>
-<instance part="C13" gate="G$1" x="167.64" y="215.9"/>
-<instance part="C14" gate="G$1" x="172.72" y="215.9"/>
-<instance part="C15" gate="G$1" x="177.8" y="215.9"/>
+<instance part="+3V7" gate="G$1" x="208.28" y="325.12" rot="MR0"/>
+<instance part="R16" gate="G$1" x="200.66" y="320.04" rot="MR180"/>
 <instance part="GND4" gate="1" x="38.1" y="20.32"/>
 <instance part="C18" gate="G$1" x="48.26" y="38.1"/>
@@
 <instance part="JP1" gate="A" x="419.1" y="134.62"/>
 <instance part="U$1" gate="G$1" x="149.86" y="363.22"/>
+<instance part="GND3" gate="1" x="190.5" y="312.42"/>
+<instance part="GND5" gate="1" x="213.36" y="378.46"/>
 </instances>
 <busses>
@@
 <pinref part="Y1" gate="G$1" pin="2"/>
 <pinref part="GND2" gate="1" pin="GND"/>
-<wire x1="317.5" y1="218.44" x2="314.96" y2="218.44" width="0.1524" layer="91"/>
-<wire x1="314.96" y1="218.44" x2="314.96" y2="215.9" width="0.1524" layer="91"/>
+<wire x1="119.38" y1="320.04" x2="116.84" y2="320.04" width="0.1524" layer="91"/>
+<wire x1="116.84" y1="320.04" x2="116.84" y2="317.5" width="0.1524" layer="91"/>
 </segment>
 <segment>
@@
 <junction x="137.16" y="210.82"/>
 <junction x="142.24" y="210.82"/>
-<junction x="147.32" y="210.82"/>
 <pinref part="GND1" gate="1" pin="GND"/>
 <wire x1="132.08" y1="208.28" x2="132.08" y2="210.82" width="0.1524" layer="91"/>
 <junction x="132.08" y="210.82"/>
-<pinref part="C15" gate="G$1" pin="2"/>
-<pinref part="C14" gate="G$1" pin="2"/>
-<wire x1="177.8" y1="210.82" x2="172.72" y2="210.82" width="0.1524" layer="91"/>
-<pinref part="C13" gate="G$1" pin="2"/>
-<wire x1="172.72" y1="210.82" x2="167.64" y2="210.82" width="0.1524" layer="91"/>
-<pinref part="C12" gate="G$1" pin="2"/>
-<wire x1="167.64" y1="210.82" x2="162.56" y2="210.82" width="0.1524" layer="91"/>
-<pinref part="C10" gate="G$1" pin="2"/>
-<wire x1="162.56" y1="210.82" x2="157.48" y2="210.82" width="0.1524" layer="91"/>
-<pinref part="C9" gate="G$1" pin="2"/>
-<wire x1="157.48" y1="210.82" x2="152.4" y2="210.82" width="0.1524" layer="91"/>
-<wire x1="152.4" y1="210.82" x2="147.32" y2="210.82" width="0.1524" layer="91"/>
-<junction x="172.72" y="210.82"/>
-<junction x="167.64" y="210.82"/>
-<junction x="162.56" y="210.82"/>
-<junction x="157.48" y="210.82"/>
-<junction x="152.4" y="210.82"/>
 </segment>
 <segment>
@@
 <junction x="167.64" y="304.8"/>
 </segment>
+<segment>
+<pinref part="U$1" gate="G$1" pin="BOOT0"/>
+<pinref part="GND3" gate="1" pin="GND"/>
+<wire x1="187.96" y1="317.5" x2="190.5" y2="317.5" width="0.1524" layer="91"/>
+<wire x1="190.5" y1="317.5" x2="190.5" y2="314.96" width="0.1524" layer="91"/>
+</segment>
+<segment>
+<pinref part="U$1" gate="G$1" pin="PB2"/>
+<pinref part="GND5" gate="1" pin="GND"/>
+<wire x1="187.96" y1="381" x2="213.36" y2="381" width="0.1524" layer="91"/>
+</segment>
 </net>
 <net name="+3V3" class="0">
@@
 <segment>
 <pinref part="+3V7" gate="G$1" pin="+3V3"/>
-<wire x1="220.98" y1="215.9" x2="200.66" y2="215.9" width="0.1524" layer="91"/>
 <pinref part="R16" gate="G$1" pin="2"/>
-<wire x1="203.2" y1="213.36" x2="200.66" y2="213.36" width="0.1524" layer="91"/>
-<wire x1="200.66" y1="213.36" x2="200.66" y2="215.9" width="0.1524" layer="91"/>
-<junction x="200.66" y="215.9"/>
+<wire x1="205.74" y1="320.04" x2="208.28" y2="320.04" width="0.1524" layer="91"/>
+<wire x1="208.28" y1="320.04" x2="208.28" y2="322.58" width="0.1524" layer="91"/>
 </segment>
 <segment>
@@
 <wire x1="132.08" y1="220.98" x2="132.08" y2="218.44" width="0.1524" layer="91"/>
 <junction x="132.08" y="218.44"/>
-<pinref part="C9" gate="G$1" pin="1"/>
-<wire x1="147.32" y1="218.44" x2="152.4" y2="218.44" width="0.1524" layer="91"/>
-<pinref part="C10" gate="G$1" pin="1"/>
-<wire x1="152.4" y1="218.44" x2="157.48" y2="218.44" width="0.1524" layer="91"/>
-<pinref part="C12" gate="G$1" pin="1"/>
-<wire x1="157.48" y1="218.44" x2="162.56" y2="218.44" width="0.1524" layer="91"/>
-<pinref part="C13" gate="G$1" pin="1"/>
-<wire x1="162.56" y1="218.44" x2="167.64" y2="218.44" width="0.1524" layer="91"/>
-<pinref part="C14" gate="G$1" pin="1"/>
-<wire x1="167.64" y1="218.44" x2="172.72" y2="218.44" width="0.1524" layer="91"/>
-<pinref part="C15" gate="G$1" pin="1"/>
-<wire x1="172.72" y1="218.44" x2="177.8" y2="218.44" width="0.1524" layer="91"/>
-<junction x="147.32" y="218.44"/>
-<junction x="152.4" y="218.44"/>
-<junction x="157.48" y="218.44"/>
-<junction x="162.56" y="218.44"/>
-<junction x="167.64" y="218.44"/>
-<junction x="172.72" y="218.44"/>
 </segment>
 <segment>
@@
 <segment>
 <pinref part="Y1" gate="G$1" pin="3"/>
-<wire x1="335.28" y1="215.9" x2="325.12" y2="215.9" width="0.1524" layer="91"/>
+<wire x1="137.16" y1="317.5" x2="127" y2="317.5" width="0.1524" layer="91"/>
+<pinref part="U$1" gate="G$1" pin="PD1-OSC_OUT"/>
+<junction x="137.16" y="317.5"/>
 </segment>
 </net>
 <net name="N$2" class="0">
 <segment>
-<wire x1="335.28" y1="218.44" x2="332.74" y2="218.44" width="0.1524" layer="91"/>
-<wire x1="332.74" y1="218.44" x2="332.74" y2="220.98" width="0.1524" layer="91"/>
+<wire x1="137.16" y1="320.04" x2="134.62" y2="320.04" width="0.1524" layer="91"/>
+<wire x1="134.62" y1="320.04" x2="134.62" y2="322.58" width="0.1524" layer="91"/>
 <pinref part="Y1" gate="G$1" pin="1"/>
-<wire x1="332.74" y1="220.98" x2="325.12" y2="220.98" width="0.1524" layer="91"/>
+<wire x1="134.62" y1="322.58" x2="127" y2="322.58" width="0.1524" layer="91"/>
+<pinref part="U$1" gate="G$1" pin="PD0-OSC_IN"/>
+<junction x="137.16" y="320.04"/>
 </segment>
 </net>
@@
 <label x="22.86" y="142.24" size="1.778" layer="95"/>
 </segment>
+<segment>
+<pinref part="U$1" gate="G$1" pin="PA13"/>
+<wire x1="137.16" y1="353.06" x2="104.14" y2="353.06" width="0.1524" layer="91"/>
+<label x="106.68" y="353.06" size="1.778" layer="95"/>
+</segment>
 </net>
 <net name="TCK" class="0">
@@
 <label x="22.86" y="139.7" size="1.778" layer="95"/>
 </segment>
+<segment>
+<pinref part="U$1" gate="G$1" pin="PA14"/>
+<wire x1="137.16" y1="350.52" x2="104.14" y2="350.52" width="0.1524" layer="91"/>
+<label x="106.68" y="350.52" size="1.778" layer="95"/>
+</segment>
 </net>
 <net name="TDO" class="0">
@@
 <label x="71.12" y="167.64" size="1.778" layer="95"/>
 </segment>
+<segment>
+<pinref part="U$1" gate="G$1" pin="PB3"/>
+<wire x1="187.96" y1="378.46" x2="208.28" y2="378.46" width="0.1524" layer="91"/>
+<label x="190.5" y="378.46" size="1.778" layer="95"/>
+</segment>
 </net>
 <net name="TRST" class="0">
@@
 <wire x1="93.98" y1="165.1" x2="68.58" y2="165.1" width="0.1524" layer="91"/>
 <label x="71.12" y="165.1" size="1.778" layer="95"/>
+</segment>
+<segment>
+<pinref part="U$1" gate="G$1" pin="PB4"/>
+<wire x1="187.96" y1="375.92" x2="208.28" y2="375.92" width="0.1524" layer="91"/>
+<label x="190.5" y="375.92" size="1.778" layer="95"/>
 </segment>
 </net>
@@
 <segment>
 <pinref part="R16" gate="G$1" pin="1"/>
-<wire x1="220.98" y1="213.36" x2="213.36" y2="213.36" width="0.1524" layer="91"/>
-<label x="213.36" y="213.36" size="1.778" layer="95"/>
-</segment>
-</net>
+<wire x1="187.96" y1="320.04" x2="195.58" y2="320.04" width="0.1524" layer="91"/>
+<label x="195.58" y="320.04" size="1.778" layer="95" rot="MR0"/>
+<pinref part="U$1" gate="G$1" pin="NRST"/>
+<junction x="187.96" y="320.04"/>
+</segment>
+</net>

Commit message: connect led matrix
Connections:
- removed net USART3_RX: FTDI.3
- removed net USART3_TX: FTDI.2
- new net NC: U$1.PC13-TAMPER-RTC
- new net USART1_RX: FTDI.3, U$1.PA10
- new net USART1_TX: FTDI.2, U$1.PA9
- net ADXL345_INT2: now also U$1.PC1
- net ARCDOZEN_1: now also U$1.PB7
- net ARCDOZEN_10: now also U$1.PB0
- net ARCDOZEN_11: now also U$1.PB1
- net ARCDOZEN_12: now also U$1.PB6
- net ARCDOZEN_2: now also U$1.PB8
- net ARCDOZEN_3: now also U$1.PB9
- net ARCDOZEN_4: now also U$1.PA0_WKUP
- net ARCDOZEN_5: now also U$1.PA1
- net ARCDOZEN_6: now also U$1.PA2
- net ARCDOZEN_7: now also U$1.PA3
- net ARCDOZEN_8: now also U$1.PC6
- net ARCDOZEN_9: now also U$1.PC7
- net LIGHT_SENSOR: now also U$1.PC0
- net N$10: now also U$1.PB13
- net N$11: now also U$1.PB14
- net N$12: now also U$1.PB15
- net N$13: now also U$1.PC9
- net N$14: now also U$1.PC8
- net N$15: now also U$1.PC12
- net N$16: now also U$1.PC11
- net N$17: now also U$1.PC10
- net N$35: now also U$1.PC5
- net N$7: now also U$1.PB10
- net N$8: now also U$1.PB11
- net N$9: now also U$1.PB12
- net SPI1_MISO: now also U$1.PA6
- net SPI1_MOSI: now also U$1.PA7
- net SPI1_NSS: now also U$1.PA4
- net SPI1_SCK: now also U$1.PA5
- net USB_DISCONNECT: now also U$1.PA8
- net USB_DM: now also U$1.PA11
- net USB_DP: now also U$1.PA12
Other:
- note added: "TIM3"
- note removed: "SPI1"
- note removed: "SPI2"
- note removed: "TIM1 remap"
- note removed: "TIM8"
- note removed: "USART3 remap"
- moved on the sheet: C6, C7, R1, R10, R11, R12, R13, R15, R2, R3, R4, R5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

Commit message: all within dimension lines
Other:
- moved on the sheet: C1, C2, C20, C3, C4, C6, C7, C8, HOUR0, HOUR1, HOUR10, HOUR11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

Commit message: Board outline and mounting
Parts:
- removed R15: 0, Custom components:R-EU_R0603
- added EXT_INTERFACE: (no value), Custom components:PINHD-2X3SMT
- added JP2: (no value), SparkFun2012:JUMPER-2SMD-NO
- added Q1: 2N7002CK4SST, Custom components:2N7002CK4SST
- C6, C7: value 100n -> 6.8p
- renumbered MASTER_PROG to PROG
Connections:
- removed net NC: U$1.PC13-TAMPER-RTC
- new net N$20: EXT_INTERFACE.4, Q1.D
- new net TOUCH1: U$1.PA15
- new net TOUCH2: U$1.PC3
- new net TOUCH3: U$1.PC4
- new net TOUCH4: U$1.PD2
- new net TOUCH5: U$1.PB5
- new net WAKE: Q1.G, U$1.PC13-TAMPER-RTC
- net +5V: now also EXT_INTERFACE.1, JP2.1; no longer U$12.VBUS
- net ADXL345_INT1: now also U$1.PC2
- net GND: now also EXT_INTERFACE.5, Q1.S
- net N$3: now also JP2.2, U$12.VBUS; no longer R15.2, U$1.PC14-OSC32_IN
- net N$5: now also U$2.P$4; no longer U$2.P$1
- net N$6: now also U$1.PC14-OSC32_IN, U$2.P$1; no longer R15.1, U$2.P$4
- net USART1_RX: now also EXT_INTERFACE.2
- net USART1_TX: now also EXT_INTERFACE.3
Other:
- moved on the sheet: C1, C2, C20, C3, C4, C6, C7, C8, FTDI, JP1, R13

Commit message: routing
Connections:
- net USART1_RX: now also EXT_INTERFACE.3; no longer EXT_INTERFACE.2
- net USART1_TX: now also EXT_INTERFACE.2; no longer EXT_INTERFACE.3
Changed lines of the file:
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@@
 </segment>
 <segment>
-<pinref part="EXT_INTERFACE" gate="A" pin="3"/>
-<wire x1="424.18" y1="142.24" x2="391.16" y2="142.24" width="0.1524" layer="91"/>
-<label x="393.7" y="142.24" size="1.778" layer="95"/>
+<pinref part="EXT_INTERFACE" gate="A" pin="2"/>
+<wire x1="431.8" y1="144.78" x2="457.2" y2="144.78" width="0.1524" layer="91"/>
+<label x="439.42" y="144.78" size="1.778" layer="95"/>
 </segment>
 </net>
@@
 </segment>
 <segment>
-<pinref part="EXT_INTERFACE" gate="A" pin="2"/>
-<wire x1="431.8" y1="144.78" x2="457.2" y2="144.78" width="0.1524" layer="91"/>
-<label x="439.42" y="144.78" size="1.778" layer="95"/>
+<pinref part="EXT_INTERFACE" gate="A" pin="3"/>
+<wire x1="424.18" y1="142.24" x2="391.16" y2="142.24" width="0.1524" layer="91"/>
+<label x="393.7" y="142.24" size="1.778" layer="95"/>
 </segment>
 </net>

Commit message: routing
Parts:
- removed C26: 100n, Custom components:C-EUC0603
Connections:
- net +3V3: no longer C26.1
- net GND: no longer C26.2
Other:
- moved on the sheet: C27
Changed lines of the file:
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@@
 <part name="U2" library="SparkFun2012" deviceset="ADXL345" device=""/>
 <part name="C5" library="Custom components" deviceset="C-EU" device="C0603" value="100n"/>
-<part name="C26" library="Custom components" deviceset="C-EU" device="C0603" value="100n"/>
 <part name="C27" library="Custom components" deviceset="C-EU" device="C0603" value="10u"/>
 <part name="+3V6" library="Custom components" deviceset="+3V3" device=""/>
@@
 <instance part="U2" gate="G$1" x="299.72" y="35.56"/>
 <instance part="C5" gate="G$1" x="284.48" y="38.1"/>
-<instance part="C26" gate="G$1" x="276.86" y="38.1"/>
-<instance part="C27" gate="G$1" x="269.24" y="38.1"/>
+<instance part="C27" gate="G$1" x="276.86" y="38.1"/>
 <instance part="+3V6" gate="G$1" x="284.48" y="50.8"/>
 <instance part="GND12" gate="1" x="284.48" y="17.78"/>
@@
 <pinref part="C27" gate="G$1" pin="2"/>
 <wire x1="284.48" y1="27.94" x2="276.86" y2="27.94" width="0.1524" layer="91"/>
-<wire x1="276.86" y1="27.94" x2="269.24" y2="27.94" width="0.1524" layer="91"/>
-<wire x1="269.24" y1="27.94" x2="269.24" y2="33.02" width="0.1524" layer="91"/>
-<pinref part="C26" gate="G$1" pin="2"/>
-<wire x1="276.86" y1="33.02" x2="276.86" y2="27.94" width="0.1524" layer="91"/>
+<wire x1="276.86" y1="27.94" x2="276.86" y2="33.02" width="0.1524" layer="91"/>
 <pinref part="C5" gate="G$1" pin="2"/>
 <wire x1="284.48" y1="33.02" x2="284.48" y2="27.94" width="0.1524" layer="91"/>
 <junction x="284.48" y="27.94"/>
-<junction x="276.86" y="27.94"/>
 <junction x="284.48" y="27.94"/>
 <junction x="284.48" y="25.4"/>
@@
 <wire x1="289.56" y1="45.72" x2="284.48" y2="45.72" width="0.1524" layer="91"/>
 <pinref part="C27" gate="G$1" pin="1"/>
-<wire x1="269.24" y1="40.64" x2="269.24" y2="43.18" width="0.1524" layer="91"/>
-<wire x1="269.24" y1="43.18" x2="276.86" y2="43.18" width="0.1524" layer="91"/>
-<pinref part="C26" gate="G$1" pin="1"/>
+<wire x1="276.86" y1="40.64" x2="276.86" y2="43.18" width="0.1524" layer="91"/>
 <wire x1="276.86" y1="43.18" x2="284.48" y2="43.18" width="0.1524" layer="91"/>
-<wire x1="276.86" y1="40.64" x2="276.86" y2="43.18" width="0.1524" layer="91"/>
 <pinref part="C5" gate="G$1" pin="1"/>
 <wire x1="284.48" y1="40.64" x2="284.48" y2="43.18" width="0.1524" layer="91"/>
-<junction x="276.86" y="43.18"/>
 <junction x="284.48" y="43.18"/>
 <junction x="284.48" y="43.18"/>
