File: uac.brd (EAGLE design)
At the start: 100 x 100 mm, 201 parts, among them Q1 2N7002CK4SST, Q6 2N7002CK4SST, Q7 2N7002CK4SST, U2 ADXL345, Y1 RESONATORSMD

Commit message: placing special
Parts:
- moved SPECIAL4 75.3 mm to (108.0, 63.0)
- moved SPECIAL0 71.9 mm to (48.0, 37.0), turned to 180 degrees
- moved SPECIAL1 71.6 mm to (46.0, 37.0), turned to 180 degrees
- moved SPECIAL11 71.0 mm to (52.0, 37.0), turned to 0 degrees
- moved SPECIAL8 55.1 mm to (57.0, 59.5), turned to 180 degrees
- moved SPECIAL5 10.1 mm to (48.0, 63.0)
- moved SPECIAL3 5.00 mm to (37.0, 50.0)
- moved SPECIAL6 3.54 mm to (52.0, 63.0)
- moved SPECIAL7 3.50 mm to (54.0, 63.0)
Routing:
- net DOZEN3: track 54.8 -> 53.1 mm
- net ARCDOZEN_3: track 81.4 -> 82.6 mm
- net ARCDOZEN_6: track 86.6 -> 85.4 mm
- net N$6: track 9.50 -> 10.3 mm
- net USART1_RX: track 72.3 -> 73.1 mm
- net ARCDOZEN_4: track 76.6 -> 77.3 mm
- net SPI1_NSS: track 11.1 -> 10.5 mm
- net USART1_TX: track 75.6 -> 76.2 mm

Commit message: special connecten almost done
Parts:
- removed SPECIAL1, SPECIAL10, SPECIAL2, SPECIAL4, SPECIAL7, SPECIAL8: (no value), Custom components:CHIPLED_0603
- moved SPECIAL9 51.9 mm to (63.0, 50.0)
- turned SPECIAL0 to 0 degrees
- turned SPECIAL5 to 0 degrees
- turned SPECIAL6 to 0 degrees
Connections:
- net ARCDOZEN_11: no longer SPECIAL10.C
- net ARCDOZEN_2: no longer SPECIAL1.C
- net ARCDOZEN_3: no longer SPECIAL2.C
- net ARCDOZEN_5: no longer SPECIAL4.C
- net ARCDOZEN_8: no longer SPECIAL7.C
- net ARCDOZEN_9: no longer SPECIAL8.C
- net DOZEN12: no longer SPECIAL1.A, SPECIAL10.A, SPECIAL2.A, SPECIAL4.A, SPECIAL7.A, SPECIAL8.A
Routing:
- net DOZEN12: track 0.00 -> 66.8 mm, vias 0 -> 4
- net ARCDOZEN_6: track 85.4 -> 94.7 mm
- net WAKE: track 100.9 -> 96.1 mm
- net ARCDOZEN_4: track 77.3 -> 81.9 mm
- net ARCDOZEN_10: track 84.0 -> 86.4 mm
- net +3V3: track 188.0 -> 189.2 mm
- net ARCDOZEN_7: track 79.2 -> 80.4 mm
- net ARCDOZEN_1: track 79.7 -> 80.8 mm
- net ARCDOZEN_12: track 83.9 -> 85.0 mm
- net ARCDOZEN_3: track 82.6 -> 83.6 mm
- net TDO: track 69.6 -> 70.3 mm
- net GND: vias 31 -> 39
