File: Hardware/uac.brd (EAGLE design)
At the start: 100 x 100 mm, 194 parts, among them Q1 2N7002CK4SST, Q6 2N7002CK4SST, Q7 2N7002CK4SST, U2 ADXL345, Y1 RESONATORSMD

Commit message: Created keep out layer for lasercut
Parts:
- HOUR0, HOUR1, HOUR10, HOUR11, HOUR2, HOUR3, HOUR4, HOUR5, HOUR6, HOUR7, HOUR8, HOUR9, MIN0, MIN1, MIN10, MIN11, MIN12, MIN13, MIN14, MIN15, MIN16, MIN17, MIN18, MIN19, MIN2, MIN20, MIN21, MIN22, MIN23, MIN24, MIN25, MIN26, MIN27, MIN28, MIN29, MIN3, MIN30, MIN31, MIN32, MIN33, MIN34, MIN35, MIN36, MIN37, MIN38, MIN39, MIN4, MIN40, MIN41, MIN42, MIN43, MIN44, MIN45, MIN46, MIN47, MIN48, MIN49, MIN5, MIN50, MIN51, MIN52, MIN53, MIN54, MIN55, MIN56, MIN57, MIN58, MIN59, MIN6, MIN7, MIN8, MIN9, SEC0, SEC1, SEC10, SEC11, SEC12, SEC13, SEC14, SEC15, SEC16, SEC17, SEC18, SEC19, SEC2, SEC20, SEC21, SEC22, SEC23, SEC24, SEC25, SEC26, SEC27, SEC28, SEC29, SEC3, SEC30, SEC31, SEC32, SEC33, SEC34, SEC35, SEC36, SEC37, SEC38, SEC39, SEC4, SEC40, SEC41, SEC42, SEC43, SEC44, SEC45, SEC46, SEC47, SEC48, SEC49, SEC5, SEC50, SEC51, SEC52, SEC53, SEC54, SEC55, SEC56, SEC57, SEC58, SEC59, SEC6, SEC7, SEC8, SEC9, SPECIAL0, SPECIAL11, SPECIAL3, SPECIAL5, SPECIAL6, SPECIAL9: device Custom components:CHIPLED_0603 -> timearc:CHIPLED_0603
- U$1: device stm32:LQFP64 -> timearc:LQFP64
- U$11: device devergy_berkelaarmrt:FLD00030 -> timearc:FLD00030
