File: Hardware/Sides/TimearcSides.brd (EAGLE design)
At the start: 86 x 50 mm, 3 parts

Commit message: Tweaked the board File.php Enclosure.skp jorrit ideas
Parts:
- moved TOUCH1 1.00 mm to (68.0, 10.0)
- moved U$3 1.00 mm to (43.0, 10.0)
Other:
- board text added: "Time Arc, Sides Armin Oonk, Jan 2016"
Changed lines of the file:
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@@
 <hole x="78" y="7" drill="3.1"/>
 <hole x="78" y="43" drill="3.1"/>
+<wire x1="19" y1="15" x2="19" y2="5" width="0.4064" layer="25" curve="180"/>
+<wire x1="68" y1="5" x2="68" y2="15" width="0.4064" layer="25" curve="180"/>
+<wire x1="19" y1="15" x2="68" y2="15" width="0.4064" layer="25"/>
+<wire x1="68" y1="5" x2="19" y2="5" width="0.4064" layer="25"/>
+<wire x1="18" y1="10" x2="22" y2="14" width="0.4064" layer="25"/>
+<wire x1="18" y1="10" x2="22" y2="6" width="0.4064" layer="25"/>
+<wire x1="53" y1="10" x2="49" y2="6" width="0.4064" layer="25"/>
+<wire x1="53" y1="10" x2="49" y2="14" width="0.4064" layer="25"/>
+<wire x1="68" y1="10" x2="64" y2="6" width="0.4064" layer="25"/>
+<wire x1="68" y1="10" x2="64" y2="14" width="0.4064" layer="25"/>
+<circle x="43" y="10" radius="4" width="0.4064" layer="25"/>
+<wire x1="23" y1="10" x2="27" y2="14" width="0.4064" layer="25"/>
+<wire x1="23" y1="10" x2="27" y2="6" width="0.4064" layer="25"/>
+<wire x1="28" y1="10" x2="32" y2="14" width="0.4064" layer="25"/>
+<wire x1="28" y1="10" x2="32" y2="6" width="0.4064" layer="25"/>
+<wire x1="33" y1="10" x2="37" y2="14" width="0.4064" layer="25"/>
+<wire x1="33" y1="10" x2="37" y2="6" width="0.4064" layer="25"/>
+<wire x1="63" y1="10" x2="59" y2="6" width="0.4064" layer="25"/>
+<wire x1="63" y1="10" x2="59" y2="14" width="0.4064" layer="25"/>
+<wire x1="58" y1="10" x2="54" y2="6" width="0.4064" layer="25"/>
+<wire x1="58" y1="10" x2="54" y2="14" width="0.4064" layer="25"/>
+<text x="56" y="44" size="1.778" layer="26" font="vector" rot="MR0">Time Arc, Sides
+Armin Oonk, Jan 2016</text>
 </plain>
 <attributes>
@@
 </autorouter>
 <elements>
-<element name="TOUCH1" library="timearc" package="SOLDER_PAD" value="SOLDER_PAD" x="69" y="10" rot="MR0"/>
+<element name="TOUCH1" library="timearc" package="SOLDER_PAD" value="SOLDER_PAD" x="68" y="10" rot="MR0"/>
 <element name="TOUCH2" library="timearc" package="SOLDER_PAD" value="SOLDER_PAD" x="18" y="10" rot="MR0"/>
-<element name="U$3" library="timearc" package="SOLDER_PAD" value="SOLDER_PAD" x="44" y="10" rot="MR0"/>
+<element name="U$3" library="timearc" package="SOLDER_PAD" value="SOLDER_PAD" x="43" y="10" rot="MR0"/>
 </elements>
 <signals>
@@
 </polygon>
 <via x="44" y="18" extent="1-16" drill="0.31"/>
-<polygon width="0.2032" layer="1" isolate="1.016" rank="2">
+<polygon width="0.2032" layer="1" isolate="0.3048" rank="2">
 <vertex x="0" y="0"/>
 <vertex x="0" y="19"/>
@@
 <signal name="TOUCH1">
 <contactref element="TOUCH1" pad="1"/>
-<via x="70" y="6" extent="1-16" drill="0.31"/>
+<via x="69" y="6" extent="1-16" drill="0.31"/>
 <polygon width="0.2032" layer="1" isolate="0.3048">
 <vertex x="71" y="14"/>
@@
 <vertex x="16" y="5"/>
 </polygon>
-<wire x1="70" y1="6" x2="70" y2="9" width="0.2032" layer="16"/>
-<wire x1="70" y1="9" x2="69" y2="10" width="0.2032" layer="16"/>
+<wire x1="69" y1="6" x2="69" y2="9" width="0.2032" layer="16"/>
+<wire x1="69" y1="9" x2="68" y2="10" width="0.2032" layer="16"/>
 </signal>
 <signal name="TOUCH2">
@@
 </board>
 </drawing>
+<compatibility>
+<note version="6.3" minversion="6.2.2" severity="warning">
+Since Version 6.2.2 text objects can contain more than one line,
+which will not be processed correctly with this version.
+</note>
+</compatibility>
 </eagle>
