File: Hardware/RPi/RPi.kicad_pcb (KiCad board)
At the start: 2 copper layers, 100 x 100 mm, 76 parts, among them P10 Solder_Pad, P11 Solder_Pad, P12 Solder_Pad, P13 Solder_Pad, P14 Solder_Pad, P15 Solder_Pad, P16 Solder_Pad, P17 Solder_Pad, P18 Solder_Pad, P19 Solder_Pad, P2 Solder_Pad, P20 Solder_Pad, P21 Solder_Pad, P3 Solder_Pad, P4 Solder_Pad, P7 Solder_Pad, P8 Solder_Pad, P9 Solder_Pad, U1 MPU_9150, U10 WS2812B, U11 WS2812B, U12 WS2812B, U13 Teensy_LC, U14 WS2812B, U15 WS2812B, U16 WS2812B, U17 WS2812B, U18 WS2812B, U19 WS2812B, U2 RPi_Interface, U20 SolderpadPowerOut, U21 SolderpadPowerOut, U4 AP1117E25, U5 Dual_buffer_NC7WZ16, U6 ESP-12E, U7 WS2812B, U8 WS2812B, U9 WS2812B

Commit message: Restructure
Parts:
- moved U6 61.4 mm to (11.5, 78.5), turned to 90 degrees
- moved C11 42.2 mm to (31.0, 79.0), turned to 0 degrees
- moved R14 39.2 mm to (31.0, 76.5), turned to 180 degrees
- moved R26 38.7 mm to (21.5, 58.5)
- moved R15 36.3 mm to (31.0, 74.0), turned to 180 degrees
- moved R16 33.6 mm to (31.0, 71.5), turned to 180 degrees
- moved R17 31.0 mm to (31.0, 69.0), turned to 180 degrees
- moved R18 28.6 mm to (31.0, 66.5), turned to 180 degrees
- moved R19 26.5 mm to (31.0, 64.0), turned to 180 degrees
- moved P14 5.00 mm to (55.0, 35.5)
- moved P15 5.00 mm to (55.0, 40.5)
- moved P16 5.00 mm to (65.0, 35.5)
- moved P19 5.00 mm to (65.0, 40.5)
- moved P7 5.00 mm to (50.0, 35.5)
- moved P8 5.00 mm to (50.0, 40.5)
Routing:
- net GND: track 0.00 -> 65.7 mm, vias 0 -> 23
- net SD_D3: track 0.00 -> 48.5 mm, vias 0 -> 2
- net SD_DO: track 0.00 -> 44.4 mm, vias 0 -> 2
- net SD_D1: track 0.00 -> 41.7 mm, vias 0 -> 2
- net SD_CMD: track 0.00 -> 40.7 mm, vias 0 -> 2
- net ID_SD: track 0.00 -> 40.0 mm
- net Net-(P19-Pad1): track 0.00 -> 33.5 mm
- net Net-(P15-Pad1): track 0.00 -> 27.8 mm
- net PWM0: track 0.00 -> 25.8 mm, vias 0 -> 2
- net Net-(P14-Pad1): track 0.00 -> 24.3 mm
- net Net-(P16-Pad1): track 0.00 -> 22.8 mm
- net SD_D2: track 0.00 -> 20.7 mm, vias 0 -> 2
- net PWM1: track 0.00 -> 19.4 mm
- net +3V3: track 0.00 -> 16.8 mm
- net Net-(P8-Pad1): track 0.00 -> 15.0 mm
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- added copper zone on B.Cu, net GND
Other:
- net class Default: clearance 0.2 -> 0.15; via_dia 0.6 -> 0.7; via_drill 0.4 -> 0.3
- rule trace_clearance: 0.2 -> 0.15
- rule via_min_size: 0.4 -> 0.25
