File: Hardware/Front2016/Front 2016.sch (EAGLE design)
At the start: 176 parts

Commit message: Connecting the seconds
Connections:
- new net N$13: ICH13.R, SEC17.C
- new net N$14: ICH9.R, SEC11.C
- new net N$15: ICH9.G, SEC12.C
- new net N$16: ICH9.B, SEC13.C
- new net N$17: ICH26.G, SEC38.C
- new net N$18: ICH10.R, SEC14.C
- new net N$19: ICH10.G, SEC15.C
- new net N$20: ICH10.B, SEC16.C
- new net N$21: ICH14.R, SEC20.C
- new net N$22: ICH13.G, SEC18.C
- new net N$23: ICH13.B, SEC19.C
- new net N$24: ICH14.G, SEC21.C
- new net N$25: ICH14.B, SEC22.C
- new net N$26: ICH26.B, SEC40.C
- new net N$27: ICH17.R, SEC23.C
- new net N$28: ICH17.G, SEC24.C
- new net N$29: ICH17.B, SEC25.C
- new net N$30: ICH18.R, SEC26.C
- new net N$31: ICH18.G, SEC27.C
- new net N$32: ICH18.B, SEC28.C
- new net N$33: ICH30.DIN
- new net N$34: ICH29.R, SEC41.C
- new net N$35: ICH21.R, SEC29.C
- new net N$36: ICH21.G, SEC31.C
- new net N$37: ICH21.B, SEC30.C
- new net N$38: ICH29.G, SEC42.C
- new net N$39: ICH22.R, SEC32.C
- new net N$40: ICH22.G, SEC33.C
- new net N$41: ICH22.B, SEC34.C
- new net N$42: ICH29.B, SEC43.C
- new net N$43: ICH25.R, SEC35.C
- new net N$44: ICH25.G, SEC36.C
- new net N$45: ICH25.B, SEC37.C
- new net N$46: ICH30.DO, ICH33.DIN
- new net N$47: ICH26.R, SEC39.C
- new net N$48: ICH30.R, SEC44.C
- new net N$49: ICH30.G, SEC45.C
- new net N$50: ICH30.B, SEC46.C
- new net N$51: ICH33.DO, ICH34.DIN
- new net N$52: ICH33.R, SEC47.C
- new net N$53: ICH33.G, SEC48.C
- new net N$54: ICH33.B, SEC49.C
- new net N$55: ICH34.DO, ICH37.DIN
- new net N$56: ICH34.R, SEC50.C
- new net N$57: ICH34.G, SEC51.C
- new net N$58: ICH34.B, SEC52.C
- new net N$59: ICH37.DO, ICH41.DIN
- new net N$60: ICH37.R, SEC53.C
- new net N$61: ICH37.G, SEC54.C
- new net N$62: ICH37.B, SEC55.C
- new net N$64: ICH41.R, SEC56.C
- new net N$65: ICH41.G, SEC57.C
- new net N$66: ICH41.B, SEC58.C
- new net N$67: ICH1.DO, ICH2.DIN
- new net N$68: ICH2.DO, ICH5.DIN
- new net N$69: ICH5.DO, ICH6.DIN
- new net N$70: ICH6.DO, ICH9.DIN
- new net N$71: ICH10.DIN, ICH9.DO
- new net N$72: ICH10.DO, ICH13.DIN
- new net N$73: ICH13.DO, ICH14.DIN
- new net N$74: ICH14.DO, ICH17.DIN
- new net N$75: ICH17.DO, ICH18.DIN
- new net N$76: ICH18.DO, ICH21.DIN
- new net N$77: ICH21.DO, ICH22.DIN
- new net N$78: ICH22.DO, ICH25.DIN
- new net N$79: ICH25.DO, ICH26.DIN
- new net N$80: ICH26.DO, ICH29.DIN
- net 5V: now also SEC11.A, SEC12.A, SEC13.A, SEC14.A, SEC15.A, SEC16.A, SEC17.A, SEC18.A, SEC19.A, SEC20.A, SEC21.A, SEC22.A, SEC23.A, SEC24.A, SEC25.A, SEC26.A, SEC27.A, SEC28.A, SEC29.A, SEC30.A, SEC31.A, SEC32.A, SEC33.A, SEC34.A, SEC35.A, SEC36.A, SEC37.A, SEC38.A, SEC39.A, SEC40.A, SEC41.A, SEC42.A, SEC43.A, SEC44.A, SEC45.A, SEC46.A, SEC47.A, SEC48.A, SEC49.A, SEC50.A, SEC51.A, SEC52.A, SEC53.A, SEC54.A, SEC55.A, SEC56.A, SEC57.A, SEC58.A
Other:
- moved on the sheet: ICH1, ICH10, ICH13, ICH14, ICH17, ICH18, ICH2, ICH21, ICH22, ICH25, ICH26, ICH29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

Commit message: Connected rest of schematic, added solderpad for +5V, DIN, DOUT, GND Added a footprint for a capacitor in the ws8211 footprint
Parts:
- added +5V, +5V1, DIN, DOUT, GND, GND46: SOLDER_PAD, timearc:SOLDER_PAD
- ICC1, ICC2, ICC3, ICC4, ICH1, ICH10, ICH13, ICH14, ICH17, ICH18, ICH2, ICH21, ICH22, ICH25, ICH26, ICH29, ICH30, ICH33, ICH34, ICH37, ICH41, ICH5, ICH6, ICH9, ICL11, ICL12, ICL15, ICL16, ICL19, ICL20, ICL23, ICL24, ICL27, ICL28, ICL3, ICL31, ICL32, ICL35, ICL36, ICL39, ICL4, ICL43, ICL7, ICL8: device adafruit:WS2811-SOP8 -> timearc:WS2811-SOP8
Connections:
- new net N$100: ICL12.G, MIN15.C
- new net N$101: ICL12.B, MIN16.C
- new net N$102: ICL11.DIN, ICL8.DO
- new net N$103: ICL15.R, MIN17.C
- new net N$104: ICL15.G, MIN18.C
- new net N$105: ICL15.B, MIN19.C
- new net N$106: ICL11.DO, ICL12.DIN
- new net N$107: ICL16.R, MIN20.C
- new net N$108: ICL16.G, MIN21.C
- new net N$109: ICL16.B, MIN22.C
- new net N$110: ICL12.DO, ICL15.DIN
- new net N$111: ICL19.R, MIN23.C
- new net N$112: ICL19.G, MIN24.C
- new net N$113: ICL19.B, MIN25.C
- new net N$114: ICL15.DO, ICL16.DIN
- new net N$115: ICL20.R, MIN26.C
- new net N$116: ICL20.G, MIN27.C
- new net N$117: ICL20.B, MIN28.C
- new net N$118: ICL16.DO, ICL19.DIN
- new net N$119: ICL23.R, MIN29.C
- new net N$120: ICL23.G, MIN30.C
- new net N$121: ICL23.B, MIN31.C
- new net N$122: ICL19.DO, ICL20.DIN
- new net N$123: ICL24.R, MIN32.C
- new net N$124: ICL24.G, MIN33.C
- new net N$125: ICL24.B, MIN34.C
- new net N$126: ICL20.DO, ICL23.DIN
- new net N$127: ICL27.R, MIN35.C
- new net N$128: ICL27.G, MIN36.C
- new net N$129: ICL27.B, MIN37.C
- new net N$130: ICL23.DO, ICL24.DIN
- new net N$131: ICL28.R, MIN38.C
- new net N$132: ICL28.G, MIN39.C
- new net N$133: ICL28.B, MIN40.C
- new net N$134: ICL24.DO, ICL27.DIN
- new net N$135: ICL31.R, MIN41.C
- new net N$136: ICL31.G, MIN42.C
- new net N$137: ICL31.B, MIN43.C
- new net N$138: ICL27.DO, ICL28.DIN
- new net N$139: ICL32.R, MIN44.C
- new net N$140: ICL32.G, MIN45.C
- new net N$141: ICL32.B, MIN46.C
- new net N$142: ICL28.DO, ICL31.DIN
- new net N$143: ICL35.R, MIN47.C
- new net N$144: ICL35.G, MIN48.C
- new net N$145: ICL35.B, MIN49.C
- new net N$146: ICL31.DO, ICL32.DIN
- new net N$147: ICL36.R, MIN50.C
- new net N$148: ICL36.G, MIN51.C
- new net N$149: ICL36.B, MIN52.C
- new net N$150: ICL32.DO, ICL35.DIN
- new net N$151: ICL39.R, MIN53.C
- new net N$152: ICL39.G, MIN54.C
- new net N$153: ICL39.B, MIN55.C
- new net N$154: ICL35.DO, ICL36.DIN
- new net N$155: ICL43.R, MIN56.C
- new net N$156: ICL43.G, MIN57.C
- new net N$157: ICL43.B, MIN58.C
- new net N$158: ICL36.DO, ICL39.DIN
- new net N$159: ICL39.DO, ICL43.DIN
- new net N$160: DIN.P$1, ICH1.DIN
- new net N$161: HOUR11.C, ICC1.R
- new net N$162: HOUR0.C, ICC1.G
- new net N$163: HOUR1.C, ICC1.B
- new net N$164: DOUT.P$1, ICC4.DO
- new net N$165: HOUR2.C, ICC2.R
- new net N$166: HOUR3.C, ICC2.G
- new net N$167: HOUR4.C, ICC2.B
- new net N$169: HOUR5.C, ICC3.R
- new net N$170: HOUR6.C, ICC3.G
- new net N$171: HOUR7.C, ICC3.B
- new net N$173: HOUR8.C, ICC4.R
- new net N$174: HOUR9.C, ICC4.G
- new net N$175: HOUR10.C, ICC4.B
- new net N$176: ICC1.DIN, ICL43.DO
- new net N$177: ICC1.DO, ICC2.DIN
- new net N$178: ICC2.DO, ICC3.DIN
- new net N$179: ICC3.DO, ICC4.DIN
- new net N$63: ICH41.DO, ICL3.DIN
- new net N$81: ICL3.R, MIN59.C
- new net N$82: ICL3.G, MIN0.C
- new net N$83: ICL3.B, MIN1.C
- new net N$84: ICL4.R, MIN2.C
- new net N$85: ICL4.G, MIN3.C
- new net N$86: ICL4.B, MIN4.C
- new net N$87: ICL7.R, MIN5.C
- new net N$88: ICL7.G, MIN6.C
- new net N$89: ICL7.B, MIN7.C
- new net N$90: ICL8.R, MIN8.C
- new net N$91: ICL8.G, MIN9.C
- new net N$92: ICL8.B, MIN10.C
- new net N$93: ICL3.DO, ICL4.DIN
- new net N$94: ICL4.DO, ICL7.DIN
- new net N$95: ICL11.R, MIN11.C
- new net N$96: ICL11.G, MIN12.C
- new net N$97: ICL11.B, MIN13.C
- new net N$98: ICL7.DO, ICL8.DIN
- new net N$99: ICL12.R, MIN14.C
- net 5V: now also +5V.P$1, +5V1.P$1, HOUR0.A, HOUR1.A, HOUR10.A, HOUR11.A, HOUR2.A, HOUR3.A, HOUR4.A, HOUR5.A, HOUR6.A, HOUR7.A, HOUR8.A, HOUR9.A, MIN0.A, MIN1.A, MIN10.A, MIN11.A, MIN12.A, MIN13.A, MIN14.A, MIN15.A, MIN16.A, MIN17.A, MIN18.A, MIN19.A, MIN2.A, MIN20.A, MIN21.A, MIN22.A, MIN23.A, MIN24.A, MIN25.A, MIN26.A, MIN27.A, MIN28.A, MIN29.A, MIN3.A, MIN30.A, MIN31.A, MIN32.A, MIN33.A, MIN34.A, MIN35.A, MIN36.A, MIN37.A, MIN38.A, MIN39.A, MIN4.A, MIN40.A, MIN41.A, MIN42.A, MIN43.A, MIN44.A, MIN45.A, MIN46.A, MIN47.A, MIN48.A, MIN49.A, MIN5.A, MIN50.A, MIN51.A, MIN52.A, MIN53.A, MIN54.A, MIN55.A, MIN56.A, MIN57.A, MIN58.A, MIN59.A, MIN6.A, MIN7.A, MIN8.A, MIN9.A
- net GND: now also GND.P$1, GND46.P$1
- net N$33: now also ICH29.DO
Other:
- moved on the sheet: HOUR0, HOUR1, HOUR10, HOUR11, HOUR2, HOUR3, HOUR4, HOUR5, HOUR6, HOUR7, HOUR8, HOUR9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
