File: Hardware/Back2016/back.sch (EAGLE design)
At the start: 84 parts, among them J1 RASPBERRYPI-40-PIN-GPIO-SMT, U3 SN74LVC2G34DCKR, U4 2.5V, U5 3.3V

Commit message: Tweaked the silk screen
Parts:
- LED1, LED10, LED11, LED12, LED2, LED3, LED4, LED5, LED6, LED7, LED8, LED9: device adafruit:WS2812B5050 -> timearc:WS2812B5050
Changed lines of the file:
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@@
 <part name="JP4" library="SparkFun-Passives" deviceset="JUMPER-PAD-2-NO" device="YES_SILK" value="JUMPER-PAD-2-NOYES_SILK"/>
 <part name="JP5" library="SparkFun-Passives" deviceset="JUMPER-PAD-2-NO" device="YES_SILK" value="JUMPER-PAD-2-NOYES_SILK"/>
-<part name="LED1" library="adafruit" deviceset="WS2812B" device="5050"/>
+<part name="LED1" library="timearc" deviceset="WS2812B" device="5050"/>
 <part name="GND18" library="SparkFun-Aesthetics" deviceset="GND" device=""/>
 <part name="SUPPLY8" library="SparkFun-Aesthetics" deviceset="5V" device=""/>
-<part name="LED2" library="adafruit" deviceset="WS2812B" device="5050"/>
+<part name="LED2" library="timearc" deviceset="WS2812B" device="5050"/>
 <part name="GND19" library="SparkFun-Aesthetics" deviceset="GND" device=""/>
 <part name="SUPPLY9" library="SparkFun-Aesthetics" deviceset="5V" device=""/>
-<part name="LED3" library="adafruit" deviceset="WS2812B" device="5050"/>
+<part name="LED3" library="timearc" deviceset="WS2812B" device="5050"/>
 <part name="GND20" library="SparkFun-Aesthetics" deviceset="GND" device=""/>
 <part name="SUPPLY10" library="SparkFun-Aesthetics" deviceset="5V" device=""/>
-<part name="LED4" library="adafruit" deviceset="WS2812B" device="5050"/>
+<part name="LED4" library="timearc" deviceset="WS2812B" device="5050"/>
 <part name="GND21" library="SparkFun-Aesthetics" deviceset="GND" device=""/>
 <part name="SUPPLY11" library="SparkFun-Aesthetics" deviceset="5V" device=""/>
-<part name="LED5" library="adafruit" deviceset="WS2812B" device="5050"/>
+<part name="LED5" library="timearc" deviceset="WS2812B" device="5050"/>
 <part name="GND22" library="SparkFun-Aesthetics" deviceset="GND" device=""/>
 <part name="SUPPLY12" library="SparkFun-Aesthetics" deviceset="5V" device=""/>
-<part name="LED6" library="adafruit" deviceset="WS2812B" device="5050"/>
+<part name="LED6" library="timearc" deviceset="WS2812B" device="5050"/>
 <part name="GND23" library="SparkFun-Aesthetics" deviceset="GND" device=""/>
 <part name="SUPPLY13" library="SparkFun-Aesthetics" deviceset="5V" device=""/>
-<part name="LED7" library="adafruit" deviceset="WS2812B" device="5050"/>
+<part name="LED7" library="timearc" deviceset="WS2812B" device="5050"/>
 <part name="GND24" library="SparkFun-Aesthetics" deviceset="GND" device=""/>
 <part name="SUPPLY14" library="SparkFun-Aesthetics" deviceset="5V" device=""/>
-<part name="LED8" library="adafruit" deviceset="WS2812B" device="5050"/>
+<part name="LED8" library="timearc" deviceset="WS2812B" device="5050"/>
 <part name="GND25" library="SparkFun-Aesthetics" deviceset="GND" device=""/>
 <part name="SUPPLY15" library="SparkFun-Aesthetics" deviceset="5V" device=""/>
-<part name="LED9" library="adafruit" deviceset="WS2812B" device="5050"/>
+<part name="LED9" library="timearc" deviceset="WS2812B" device="5050"/>
 <part name="GND26" library="SparkFun-Aesthetics" deviceset="GND" device=""/>
 <part name="SUPPLY16" library="SparkFun-Aesthetics" deviceset="5V" device=""/>
-<part name="LED10" library="adafruit" deviceset="WS2812B" device="5050"/>
+<part name="LED10" library="timearc" deviceset="WS2812B" device="5050"/>
 <part name="GND27" library="SparkFun-Aesthetics" deviceset="GND" device=""/>
 <part name="SUPPLY17" library="SparkFun-Aesthetics" deviceset="5V" device=""/>
-<part name="LED11" library="adafruit" deviceset="WS2812B" device="5050"/>
+<part name="LED11" library="timearc" deviceset="WS2812B" device="5050"/>
 <part name="GND28" library="SparkFun-Aesthetics" deviceset="GND" device=""/>
 <part name="SUPPLY18" library="SparkFun-Aesthetics" deviceset="5V" device=""/>
-<part name="LED12" library="adafruit" deviceset="WS2812B" device="5050"/>
+<part name="LED12" library="timearc" deviceset="WS2812B" device="5050"/>
 <part name="GND29" library="SparkFun-Aesthetics" deviceset="GND" device=""/>
 <part name="SUPPLY19" library="SparkFun-Aesthetics" deviceset="5V" device=""/>

Commit message: Fixed stupid error in schematic
Connections:
- net ID_SD: now also U2.CH_PD; no longer U2.ADC
Changed lines of the file:
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@@
 </segment>
 <segment>
-<pinref part="U2" gate="G$1" pin="ADC"/>
-<wire x1="160.02" y1="106.68" x2="157.48" y2="106.68" width="0.1524" layer="91"/>
-<label x="157.48" y="106.68" size="1.778" layer="95" rot="R180" xref="yes"/>
+<wire x1="160.02" y1="104.14" x2="157.48" y2="104.14" width="0.1524" layer="91"/>
+<label x="157.48" y="104.14" size="1.778" layer="95" rot="R180" xref="yes"/>
+<pinref part="U2" gate="G$1" pin="CH_PD"/>
+<junction x="160.02" y="104.14"/>
 </segment>
 </net>
